File: pcb/gtxl/MAU.kicad_sch (KiCad schematic)
At the start: 5 parts, among them U10 74LS157, U12 74HCT138, U7 74LS157, U8 74LS157, U9 74LS157

Commit message: Update schematic with removed timer.  Update video timing notes.
Parts:
- removed U7, U8: 74LS157, symbol 74xx:74LS157
- added RN1: R_Network08_US, Resistor_THT:R_Array_SIP9, symbol Device:R_Network08_US
- added U47, U7, U8: 74HCT244, symbol 74xx:74HCT244
Connections:
- net +5V: now also U47.20 (VCC), U7.20 (VCC), U8.20 (VCC)
- net ADDR0: now also RN1.9 (R8), U47.18 (1Y0), U7.18 (1Y0), U8.18 (1Y0)
- net ADDR1: now also RN1.8 (R7), U47.16 (1Y1), U7.16 (1Y1), U8.16 (1Y1)
- net ADDR2: now also RN1.7 (R6), U47.14 (1Y2), U7.14 (1Y2), U8.14 (1Y2)
- net ADDR3: now also RN1.6 (R5), U47.12 (1Y3), U7.12 (1Y3), U8.12 (1Y3)
- net ADDR4: now also RN1.5 (R4), U47.3 (2Y0), U7.3 (2Y0), U8.3 (2Y0)
- net ADDR5: now also RN1.4 (R3), U47.5 (2Y1), U7.5 (2Y1), U8.5 (2Y1)
- net ADDR6: now also RN1.3 (R2), U47.7 (2Y2), U7.7 (2Y2), U8.7 (2Y2)
- net ADDR7: now also RN1.2 (R1), U47.9 (2Y3), U7.9 (2Y3), U8.9 (2Y3)
- net GND: now also RN1.1 (common), U47.10 (GND), U7.10 (GND), U8.10 (GND)
- net PC0: now also U7.2 (1A0)
- net PC1: now also U7.4 (1A1)
- net PC2: now also U7.6 (1A2)
- net PC3: now also U7.8 (1A3)
- net PC4: now also U7.17 (2A0)
- net PC5: now also U7.15 (2A1)
- net PC6: now also U7.13 (2A2)
- net PC7: now also U7.11 (2A3)
- net X0: now also U8.2 (1A0)
- net X1: now also U8.4 (1A1)
- net X2: now also U8.6 (1A2)
- net X3: now also U8.8 (1A3)
- net X4: now also U8.17 (2A0)
- net X5: now also U8.15 (2A1)
- net X6: now also U8.13 (2A2)
- net X7: now also U8.11 (2A3)
- new net DREG0: U47.2 (1A0)
- new net DREG1: U47.4 (1A1)
- new net DREG2: U47.6 (1A2)
- new net DREG3: U47.8 (1A3)
- new net DREG4: U47.17 (2A0)
- new net DREG5: U47.15 (2A1)
- new net DREG6: U47.13 (2A2)
- new net DREG7: U47.11 (2A3)
- new net EXECUTE: U7.1 (1OE), U7.19 (2OE)
- new net /IMM_MEM_EN: U47.1 (1OE), U47.19 (2OE)
- new net /XMEM_EN: U8.1 (1OE), U8.19 (2OE)
