File: pcb/gtxl/PC.kicad_sch (KiCad schematic)
At the start: 6 parts, among them U1 74LS161, U2 74LS161, U3 74LS161, U4 74LS161, U5 74LS574, U6 74LS574

Commit message: Update schematic with removed timer.  Update video timing notes.
Connections:
- net INT_EN_CLK renamed INTERRUPT
Changed lines of the file:
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@@
 		)
 	)
-	(global_label "INT_EN_CLK"
+	(global_label "INTERRUPT"
 		(shape input)
 		(at 105.41 214.63 180)
@@
 		)
 		(property "Intersheetrefs" "${INTERSHEET_REFS}"
-			(at 91.5391 214.63 0)
+			(at 92.2648 214.63 0)
 			(effects
 				(font
