File: pcb/gtxl/REGS.kicad_sch (KiCad schematic)
At the start: 15 parts, among them U19 74LS377, U20 74HCT244, U21 74LS574, U22 74HCT244, U23 74LS161, U24 74LS161, U25 74LS377

Commit message: Update schematic with removed timer.  Update video timing notes.
Parts:
- removed R10, R11, R5, R6, R7, R8, R9: 10K, symbol Device:R_US
- added RN2: R_Network08_US, Resistor_THT:R_Array_SIP9, symbol Device:R_Network08_US
- added U42: 74LS377, symbol 74xx:74LS377
Connections:
- net AC0: now also U42.3 (D0)
- net AC1: now also U42.4 (D1)
- net AC2: now also U42.7 (D2)
- net AC3: now also U42.8 (D3)
- net AC4: now also U42.13 (D4)
- net AC5: now also U42.14 (D5)
- net AC6: now also U42.17 (D6)
- net AC7: now also U42.18 (D7)
- net GND: now also RN2.1 (common)
- net VID6: now also U42.11 (CP)
- net Y0: now also RN2.8 (R7)
- net Y1: now also RN2.7 (R6)
- net Y2: now also RN2.6 (R5)
- net Y3: now also RN2.5 (R4)
- net Y4: now also RN2.4 (R3)
- net Y5: now also RN2.3 (R2)
- net Y6: now also RN2.2 (R1)
- net INTERRUPT: now reaches U24.15 (TC)
- net XCOUNT renamed EXECUTE
- new net AUDIO0: U42.2 (Q0)
- new net AUDIO1: U42.5 (Q1)
- new net AUDIO2: U42.6 (Q2)
- new net AUDIO3: U42.9 (Q3)
- new net AUDIO4: U42.12 (Q4)
- new net AUDIO5: U42.15 (Q5)
- new net AUDIO6: U42.16 (Q6)
- new net AUDIO7: U42.19 (Q7)
Other:
- moved on the sheet: R4
