File: pcb/gtxl/TIMER.kicad_sch (KiCad schematic)
At the start: 5 parts, among them U26 74LS161, U27 74LS161, U28 74LS32, U29 74LS109, U31 74LS32

Commit message: Update schematic with removed timer.  Update video timing notes.
Parts:
- removed U26, U27: 74LS161, symbol 74xx:74LS161
- removed U28, U31: 74LS32, symbol 74xx:74LS32
- removed U29: 74LS109, symbol 74xx:74LS109
Other:
- note removed: "Interrupt Enable Register"
- note removed: "Timer $4000-$4FFF"
